Commit message: add lidar

File: 03-NUCIntel/ros2_ws/src/my_robot_bringup/urdf/my_robot.xacro (robot description, xacro)
@@ -181,3 +181,24 @@
         </inertial>
       </link>
+    <joint name="laser_joint" type="fixed">
+      <parent link="base_link"/>
+      <child link="laser"/>
+      <origin xyz="0.100 0.0 0.100 " rpy="0 0 0"/>
+    </joint>
+    <!-- caster left wheel Link -->
+    <link name="laser">
+      <collision>
+        <origin xyz="0 0 0" rpy="0 0 0"/>
+        <geometry>
+	        <box size="0.040 0.040 0.080"/>
+        </geometry>
+      </collision>
+      <visual>
+        <origin xyz="0 0 0" rpy="0 0 0"/>
+        <geometry>
+		<box size="0.040 0.040 0.080"/>
+        </geometry>
+        <material name="black"/>
+      </visual>
+      </link>
 </robot>

Commit message: update config files for new robot frame

File: 03-NUCIntel/ros2_ws/src/my_robot_bringup/urdf/my_robot.xacro (robot description, xacro)
@@ -5,5 +5,5 @@
   <xacro:property name="base_mass"   value="1.0" /> <!-- arbitrary value for base mass -->
   <xacro:property name="base_width"  value="0.50" />
-  <xacro:property name="base_length" value="0.65" />
+  <xacro:property name="base_length" value="0.44" />
   <xacro:property name="base_height" value="0.04" />
   <xacro:property name="wheel_mass"  value="0.50" /> <!-- arbitrary value for wheel mass -->
@@ -14,5 +14,5 @@
   <xacro:property name="caster_wheel_mass" value="0.1" /> <!-- arbitrary value for caster wheel mass -->
   <xacro:property name="caster_wheel_radius" value="0.025" />
-  <xacro:property name="caster_x_offset" value="-0.250" />
+  <xacro:property name="caster_x_offset" value="-0.150" />
   <xacro:property name="caster_y_offset" value="0.200" />
   <xacro:property name="caster_z_offset" value="-0.010" />
@@ -184,5 +184,5 @@
       <parent link="base_link"/>
       <child link="laser"/>
-      <origin xyz="0.100 0.0 0.100 " rpy="0 0 0"/>
+      <origin xyz="-0.200 0.0 0.320 " rpy="0 0 0"/>
     </joint>
     <!-- caster left wheel Link -->

Commit message: fixing robot model new robot frame

File: 03-NUCIntel/ros2_ws/src/my_robot_bringup/urdf/my_robot.xacro (robot description, xacro)
@@ -7,5 +7,5 @@
   <xacro:property name="base_length" value="0.44" />
   <xacro:property name="base_height" value="0.04" />
-  <xacro:property name="wheel_mass"  value="0.50" /> <!-- arbitrary value for wheel mass -->
+  <xacro:property name="wheel_mass"  value="1.50" /> <!-- arbitrary value for wheel mass -->
   <xacro:property name="wheel_len"   value="0.050" />
   <xacro:property name="wheel_radius" value="0.085" />
@@ -15,6 +15,10 @@
   <xacro:property name="caster_wheel_radius" value="0.025" />
   <xacro:property name="caster_x_offset" value="-0.150" />
-  <xacro:property name="caster_y_offset" value="0.200" />
   <xacro:property name="caster_z_offset" value="-0.010" />
+  <xacro:macro name="cylinder_inertia" params="m r h">
+    <inertia  ixx="${m*(3*r*r+h*h)/12}" ixy = "0" ixz = "0"
+              iyy="${m*(3*r*r+h*h)/12}" iyz = "0"
+              izz="${m*r*r/2}" />
+  </xacro:macro>
 	<material name="white">
    		<color rgba="0.8 0.8 0.8 1"/>
@@ -86,10 +90,7 @@
         <origin xyz="0 0 0" rpy="${PI/2} 0 0"/>
         <mass value="${wheel_mass}"/>
-        <inertia
-          ixx="${wheel_mass / 12.0 * (3*wheel_radius + wheel_len*wheel_len)}" ixy="0.0" ixz="0.0"
-          iyy="${wheel_mass / 12.0 * wheel_radius*wheel_radius}" iyz="0.0"
-          izz="${wheel_mass / 12.0 * wheel_radius*wheel_radius}"/>
-        </inertial>
-      </link>
+        <xacro:cylinder_inertia  m="${wheel_mass}" r="${wheel_radius}" h="${wheel_len}" />
+      </inertial>
+    </link>
     <joint name="right_wheel_joint" type="continuous">
       <parent link="base_link"/>
@@ -117,46 +118,14 @@
         <origin xyz="0 0 0" rpy="${PI/2} 0 0"/>
         <mass value="${wheel_mass}"/>
-        <inertia
-          ixx="${wheel_mass / 12.0 * (3*wheel_radius + wheel_len*wheel_len)}" ixy="0.0" ixz="0.0"
-          iyy="${wheel_mass / 12.0 * wheel_radius*wheel_radius}" iyz="0.0"
-          izz="${wheel_mass / 12.0 * wheel_radius*wheel_radius}"/>
-        </inertial>
-      </link>
-    <joint name="caster_left_wheel_joint" type="fixed">
+        <xacro:cylinder_inertia  m="${wheel_mass}" r="${wheel_radius}" h="${wheel_len}" />
+      </inertial>
+    </link>
+    <joint name="caster_wheel_joint" type="fixed">
       <parent link="base_link"/>
-      <child link="caster_left__wheel"/>
-      <origin xyz="${caster_x_offset} ${caster_y_offset} ${caster_z_offset}" rpy="0 0 0"/>
+      <child link="caster_wheel"/>
+      <origin xyz="${caster_x_offset} 0 ${caster_z_offset}" rpy="0 0 0"/>
     </joint>
-    <joint name="caster_right_wheel_joint" type="fixed">
-      <parent link="base_link"/>
-      <child link="caster_right_wheel"/>
-      <origin xyz="${caster_x_offset} ${-caster_y_offset} ${caster_z_offset}" rpy="0 0 0"/>
-    </joint>
-    <!-- caster left wheel Link -->
-    <link name="caster_left__wheel">
-      <collision>
-        <origin xyz="0 0 0" rpy="0 0 0"/>
-        <geometry>
-          <sphere radius="${caster_wheel_radius}"/>
-        </geometry>
-      </collision>
-      <visual>
-        <origin xyz="0 0 0" rpy="0 0 0"/>
-        <geometry>
-          <sphere radius="${caster_wheel_radius}"/>
-        </geometry>
-        <material name="black"/>
-      </visual>
-      <inertial>
-        <origin xyz="0 0 0" rpy="0 0 0"/>
-        <mass value="${caster_wheel_mass}"/>
-        <inertia
-          ixx="${caster_wheel_mass * 0.4 * (caster_wheel_radius * caster_wheel_radius)}" ixy="0.0" ixz="0.0"
-          iyy="${caster_wheel_mass * 0.4 * (caster_wheel_radius * caster_wheel_radius)}" iyz="0.0"
-          izz="${caster_wheel_mass * 0.4 * (caster_wheel_radius * caster_wheel_radius)}"/>
-        </inertial>
-      </link>
-    <!-- caster right wheel Link -->
-    <link name="caster_right_wheel">
+    <!-- caster wheel Link -->
+    <link name="caster_wheel">
       <collision>
         <origin xyz="0 0 0" rpy="0 0 0"/>

Commit message: localization fix but imu yaw pb

File: 03-NUCIntel/ros2_ws/src/my_robot_bringup/urdf/my_robot.xacro (robot description, xacro)
@@ -150,5 +150,5 @@
       <parent link="base_link"/>
       <child link="laser"/>
-      <origin xyz="-0.200 0.0 0.320 " rpy="0 0 0"/>
+      <origin xyz="0.200 0.0 0.200 " rpy="0 0 0"/>
     </joint>
     <!-- laser Link -->
