Commit message: robot localization first try

File: 03-NUCIntel/ros2_ws/src/my_robot_bringup/urdf/my_robot.urdf (robot description, URDF)
Before this commit: robot my_robot, 7 links, 6 joints
Links:
- removed link world
- added link imu; collision box size=0.040 0.040 0.020; visual box size=0.040 0.040 0.020
Joints:
- removed joint worl_joint
- added joint imu_joint: type fixed, parent base_link, child imu, origin xyz=0.15 0.0 0.0  rpy=0 0 0

File: 03-NUCIntel/ros2_ws/src/my_robot_bringup/urdf/my_robot.xacro (robot description, xacro)
@@ -27,10 +27,4 @@
    		<color rgba="0.1 0.1 0.1 1"/>
    	</material>
-  <!-- ****************** ROBOT BASE FOOTPRINT ***************************  -->
-  <link name="world"/>
-  <joint name="worl_joint" type="fixed">
-    <parent link="world"/>
-    <child link="base_link"/>
-  </joint>
   <!-- ********************** ROBOT BASE *********************************  -->
   <!-- Base Link -->
@@ -65,4 +59,5 @@
     <origin xyz="0 0 ${wheel_z_offset-wheel_radius}" rpy="0 0 0"/>
   </joint>
+  <!-- ****************** ROBOT WHEELS ***************************  -->
     <joint name="left_wheel_joint" type="continuous">
       <parent link="base_link"/>
@@ -150,4 +145,6 @@
         </inertial>
       </link>
+  <!-- ****************** LASER SENSOR ***************************  -->
+    <!-- laser joint -->
     <joint name="laser_joint" type="fixed">
       <parent link="base_link"/>
@@ -155,5 +152,5 @@
       <origin xyz="-0.200 0.0 0.320 " rpy="0 0 0"/>
     </joint>
-    <!-- caster left wheel Link -->
+    <!-- laser Link -->
     <link name="laser">
       <collision>
@@ -171,3 +168,26 @@
       </visual>
       </link>
+  <!-- ****************** IMU SENSOR ***************************  -->
+  <!-- imu joint -->
+  <joint name="imu_joint" type="fixed">
+    <parent link="base_link"/>
+    <child link="imu"/>
+    <origin xyz="${wheel_x_offset} 0.0 0.0 " rpy="0 0 0"/>
+  </joint>
+  <!-- imu Link -->
+  <link name="imu">
+    <collision>
+      <origin xyz="0 0 0" rpy="0 0 0"/>
+      <geometry>
+        <box size="0.040 0.040 0.020"/>
+      </geometry>
+    </collision>
+    <visual>
+      <origin xyz="0 0 0" rpy="0 0 0"/>
+      <geometry>
+        <box size="0.040 0.040 0.020"/>
+      </geometry>
+      <material name="black"/>
+    </visual>
+  </link>
 </robot>

Commit message: urdf fix lidar new position

File: 03-NUCIntel/ros2_ws/src/my_robot_bringup/urdf/my_robot.urdf (robot description, URDF)
Before this commit: robot my_robot, 7 links, 6 joints
Joints:
- joint laser_joint: origin xyz=-0.200 0.0 0.320  rpy=0 0 0 -> xyz=0.200 0.0 0.200  rpy=0 0 0

Commit message: urdf new imu position, hb driver pkg need a better twist and pose covariance for EKF

File: 03-NUCIntel/ros2_ws/src/my_robot_bringup/urdf/my_robot.urdf (robot description, URDF)
Before this commit: robot my_robot, 7 links, 6 joints
Joints:
- joint imu_joint: origin xyz=0.15 0.0 0.0  rpy=0 0 0 -> xyz=-0.120 0.110 0.260  rpy=0 0 0
- joint laser_joint: origin xyz=0.200 0.0 0.200  rpy=0 0 0 -> xyz=0.180 0.0 0.220  rpy=0 0 0

File: 03-NUCIntel/ros2_ws/src/my_robot_bringup/urdf/my_robot.xacro (robot description, xacro)
@@ -150,5 +150,5 @@
       <parent link="base_link"/>
       <child link="laser"/>
-      <origin xyz="0.200 0.0 0.200 " rpy="0 0 0"/>
+      <origin xyz="0.180 0.0 0.220 " rpy="0 0 0"/>
     </joint>
     <!-- laser Link -->
@@ -173,5 +173,5 @@
     <parent link="base_link"/>
     <child link="imu"/>
-    <origin xyz="${wheel_x_offset} 0.0 0.0 " rpy="0 0 0"/>
+    <origin xyz="-0.120 0.110 0.260 " rpy="0 0 0"/>
   </joint>
   <!-- imu Link -->
